File: semCNC.kicad_pcb (KiCad board)
At the start: 2 copper layers, 134 parts, among them P1 UART_HEAD, P10 CONN_01X05, P11 CONN_01X03, P12 CONN_02X08, P13 CONN_01X05, P14 CONN_01X03, P15 CONN_02X08, P16 CONN_01X05, P17 CONN_01X03, P18 CONN_02X08, P19 POWER_HEAD, P2 LPT port, P3 PROG_HEAD, P4 EXPANDER PAD, P5 CONN_01X02, P6 CONN_01X02, P7 CONN_01X05, P8 CONN_01X03, P9 CONN_02X08, T1 TRANSFO, U1 MSP430G2452, U2 TIdac08s085, U3 LD1117S33CTR, U4 SPX2920U-3.3, U5 DRV8825, U6 DRV8825, U7 DRV8825, U8 DRV8825

Commit message: some modifications, before creating an array
Parts:
- moved RV4 49.7 mm to (421.6, 63.5), turned to 180 degrees
- moved C32 36.7 mm to (434.3, 83.8), turned to 0 degrees
- moved P18 34.3 mm to (397.5, 68.6), turned to 0 degrees
- moved P16 33.0 mm to (448.3, 64.8), turned to 0 degrees
- moved D5 27.0 mm to (414.0, 77.5), turned to 90 degrees
- moved P17 10.2 mm to (432.1, 66.0), turned to 180 degrees
Connections:
- D2 pad 2: /DRIVER1/3.3Vlocal -> 3.3V
- D3 pad 2: /DRIVER2/3.3Vlocal -> 3.3V
- D4 pad 2: /DRIVER3/3.3Vlocal -> 3.3V
- D5 pad 2: /DRIVER4/3.3Vlocal -> 3.3V
Routing:
- net /DRIVER4/nHOME: track 16.0 -> 76.0 mm
- net 3.3V: track 0.00 -> 59.8 mm
- net /DRIVER4/MODE2: track 15.6 -> 70.6 mm
- net /DRIVER4/MODE1: track 15.6 -> 66.5 mm
- net /DRIVER4/MODE0: track 15.8 -> 59.2 mm
- net /DRIVER4/DIR: track 0.00 -> 43.3 mm, vias 0 -> 2
- net /DRIVER4/CURR_REF: track 0.00 -> 42.2 mm
- net /DRIVER4/nENBL: track 15.5 -> 52.3 mm
- net /DRIVER4/DECAY: track 15.1 -> 48.6 mm
- net /DRIVER4/STEP: track 0.00 -> 30.8 mm, vias 0 -> 2
- net /DRIVER4/nSLEEP: track 14.2 -> 44.1 mm
- net /DRIVER4/nRESET: track 14.4 -> 41.2 mm
- net Net-(P17-Pad2): track 5.07 -> 30.4 mm, vias 0 -> 1
- net (no net): track 15.5 -> 0.00 mm
- net /DRIVER4/AOUT1: track 35.2 -> 47.4 mm
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
Commit message: Second driver
Parts:
- moved R31 369.2 mm to (525.0, 82.3)
- moved P10 365.7 mm to (530.6, 58.9)
- moved U6 331.9 mm to (502.4, 86.1), turned to 90 degrees
- moved R32 331.2 mm to (524.9, 77.7)
- moved C21 327.4 mm to (512.0, 89.7)
- moved P12 326.7 mm to (477.5, 63.0)
- moved R30 323.9 mm to (511.8, 92.7), turned to 180 degrees
- moved C20 322.3 mm to (520.2, 90.6), turned to 270 degrees
- moved P11 321.2 mm to (514.4, 61.2), turned to 180 degrees
- moved RV2 318.7 mm to (503.9, 59.2), turned to 180 degrees
- moved C18 314.1 mm to (511.8, 95.8)
- moved R33 314.0 mm to (489.0, 73.7), turned to 180 degrees
- moved C19 309.3 mm to (516.4, 73.7)
- moved D3 309.2 mm to (475.7, 76.5), turned to 90 degrees
- moved R35 307.0 mm to (489.0, 76.7), turned to 180 degrees
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Routing:
- net 3.3V: track 59.8 -> 169.2 mm, vias 0 -> 2
- net /DRIVER2/nHOME: track 0.00 -> 67.3 mm, vias 0 -> 1
- net /DRIVER2/MODE2: track 0.00 -> 60.7 mm, vias 0 -> 1
- net /DRIVER2/nFAULT: track 0.00 -> 57.2 mm, vias 0 -> 1
- net /DRIVER2/MODE1: track 0.00 -> 50.1 mm, vias 0 -> 1
- net /DRIVER2/MODE0: track 0.00 -> 45.1 mm, vias 0 -> 1
- net /DRIVER2/DIR: track 0.00 -> 41.9 mm, vias 0 -> 1
- net /DRIVER2/nENBL: track 0.00 -> 39.2 mm, vias 0 -> 1
- net /DRIVER2/DECAY: track 0.00 -> 36.4 mm, vias 0 -> 1
- net /DRIVER2/STEP: track 0.00 -> 34.5 mm, vias 0 -> 1
- net VMOT: track 45.7 -> 78.0 mm
- net /DRIVER2/nSLEEP: track 0.00 -> 26.5 mm, vias 0 -> 1
- net /DRIVER2/nRESET: track 0.00 -> 25.8 mm
- net Net-(P11-Pad2): track 0.00 -> 17.4 mm
- net GND: track 9.75 -> 27.0 mm
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
Commit message: new try to commit
Parts:
- moved C20 4.89 mm to (515.5, 89.4), turned to 90 degrees
- moved C18 3.75 mm to (508.2, 94.8)
- moved C21 3.67 mm to (508.5, 88.8)
- moved R30 3.67 mm to (508.3, 91.8)
- moved C19 2.29 mm to (517.4, 71.6), turned to 90 degrees
Routing:
- net /DRIVER2/AOUT1: track 0.00 -> 51.2 mm, vias 0 -> 1
- net /DRIVER2/AOUT2: track 6.60 -> 45.4 mm
- net /DRIVER2/BOUT2: track 8.11 -> 35.1 mm
- net VMOT: track 78.0 -> 94.1 mm
- net GND: track 27.0 -> 14.9 mm
- net Net-(R32-Pad1): track 10.7 -> 0.00 mm
- net Net-(P11-Pad2): track 17.4 -> 26.5 mm, vias 0 -> 1
- net Net-(C21-Pad2): track 8.75 -> 5.11 mm
- net /DRIVER2/nRESET: track 25.8 -> 27.8 mm, vias 0 -> 1
- net Net-(R31-Pad1): track 11.3 -> 12.6 mm
- net Net-(C21-Pad1): track 4.54 -> 3.56 mm
- net Net-(C18-Pad1): track 15.4 -> 14.8 mm

Commit message: before test
Parts:
- moved R43 240.2 mm to (343.1, 188.6)
- moved R44 240.2 mm to (384.1, 156.6)
- moved R46 240.2 mm to (403.4, 155.1)
- moved R47 240.2 mm to (396.2, 168.5)
- moved R48 240.2 mm to (403.4, 161.8)
- moved R51 240.2 mm to (375.9, 191.7)
- moved R52 240.2 mm to (387.8, 178.4)
- moved RV3 240.2 mm to (372.8, 161.7)
- moved C23 240.2 mm to (396.3, 155.1)
- moved C24 240.2 mm to (373.7, 185.0)
- moved C25 240.2 mm to (389.1, 165.0)
- moved C26 240.2 mm to (373.7, 178.3)
- moved C27 240.2 mm to (361.8, 190.4)
- moved D4 240.2 mm to (353.5, 188.8)
- moved P14 240.2 mm to (380.5, 167.8)
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Routing:
- net 3.3V: track 169.2 -> 137.7 mm
- net /DRIVER2/BOUT1: track 0.00 -> 27.7 mm, vias 0 -> 1
- net Net-(D3-Pad1): track 13.6 -> 0.00 mm
- net Net-(R32-Pad1): track 0.00 -> 10.4 mm
- net /DRIVER2/AOUT1: track 51.2 -> 55.7 mm
- net /DRIVER2/nRESET: track 27.8 -> 31.1 mm
- net VMOT: track 94.1 -> 97.3 mm
- net /DRIVER2/STEP: track 34.5 -> 32.0 mm
- net GND: track 14.9 -> 13.1 mm
- net /DRIVER2/BOUT2: track 35.1 -> 34.3 mm
- net Net-(P11-Pad1): track 8.08 -> 8.80 mm
- net /DRIVER2/nFAULT: track 57.2 -> 56.5 mm

Commit message: viktor rendberak mindent
Parts:
- moved R43 184.2 mm to (521.9, 144.3)
- moved P13 173.0 mm to (519.8, 117.8)
- moved D4 154.8 mm to (496.6, 129.8), turned to 90 degrees
- moved C24 153.7 mm to (517.4, 130.5), turned to 90 degrees
- moved C27 151.6 mm to (502.6, 134.3)
- moved U7 144.7 mm to (499.6, 146.6), turned to 90 degrees
- moved P15 143.1 mm to (467.9, 121.4)
- moved R44 138.8 mm to (521.9, 139.8)
- moved C26 134.9 mm to (505.6, 150.3)
- moved P14 131.9 mm to (503.9, 121.0), turned to 180 degrees
- moved RV3 128.2 mm to (493.4, 118.0), turned to 180 degrees
- moved C25 125.2 mm to (513.5, 150.5), turned to 90 degrees
- moved R49 123.8 mm to (481.9, 141.3), turned to 180 degrees
- moved R42 117.5 mm to (505.6, 156.3), turned to 180 degrees
- moved R51 114.9 mm to (481.9, 147.3), turned to 180 degrees
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Routing:
- net 3.3V: track 137.7 -> 403.7 mm, vias 2 -> 1
- net /DRIVER2/CURR_REF: track 0.00 -> 78.8 mm
- net VMOT: track 97.3 -> 175.0 mm
- net /DRIVER3/CURR_REF: track 0.00 -> 70.8 mm
- net /DRIVER3/nHOME: track 0.00 -> 61.9 mm, vias 0 -> 1
- net /DRIVER3/nFAULT: track 0.00 -> 61.1 mm, vias 0 -> 1
- net /DRIVER3/MODE2: track 0.00 -> 55.9 mm, vias 0 -> 1
- net /DRIVER3/MODE1: track 0.00 -> 50.4 mm, vias 0 -> 1
- net /DRIVER3/AOUT1: track 0.00 -> 46.1 mm, vias 0 -> 1
- net /DRIVER3/MODE0: track 0.00 -> 45.9 mm, vias 0 -> 1
- net /DRIVER3/DIR: track 0.00 -> 44.0 mm, vias 0 -> 1
- net /DRIVER3/nENBL: track 0.00 -> 39.5 mm, vias 0 -> 1
- net Net-(D4-Pad1): track 0.00 -> 36.9 mm, vias 0 -> 2
- net /DRIVER3/DECAY: track 0.00 -> 36.8 mm, vias 0 -> 1
- net /DRIVER3/AOUT2: track 0.00 -> 36.2 mm, vias 0 -> 1
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
Commit message: nyegyedik driver
Parts:
- moved R19 410.6 mm to (438.7, 151.0)
- moved P7 398.1 mm to (435.7, 120.2)
- moved U5 372.9 mm to (416.1, 153.5), turned to 90 degrees
- moved D2 372.3 mm to (411.2, 132.5), turned to 90 degrees
- moved R20 372.0 mm to (438.7, 146.3)
- moved C16 368.8 mm to (422.3, 157.6)
- moved C15 366.2 mm to (431.2, 157.9), turned to 90 degrees
- moved C13 361.9 mm to (422.3, 160.6)
- moved C14 361.6 mm to (434.5, 137.6), turned to 90 degrees
- moved P9 360.7 mm to (383.6, 124.4)
- moved RV1 355.6 mm to (413.6, 120.2)
- moved P8 353.6 mm to (419.5, 117.0)
- moved C17 353.2 mm to (418.9, 140.6)
- moved R29 346.7 mm to (392.9, 160.6), turned to 180 degrees
- moved R18 338.6 mm to (422.3, 163.7), turned to 180 degrees
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Routing:
- net /DRIVER1/nRESET: track 0.00 -> 25.3 mm
- net /DRIVER1/nHOME: track 0.00 -> 24.4 mm
- net /DRIVER1/nSLEEP: track 0.00 -> 24.3 mm
- net /DRIVER1/MODE2: track 0.00 -> 23.4 mm
- net /DRIVER1/nFAULT: track 0.00 -> 23.3 mm
- net /DRIVER1/MODE1: track 0.00 -> 22.5 mm
- net /DRIVER1/DECAY: track 0.00 -> 22.3 mm
- net /DRIVER1/nENBL: track 0.00 -> 21.6 mm
- net /DRIVER1/MODE0: track 0.00 -> 21.5 mm
- net /DRIVER1/DIR: track 0.00 -> 15.2 mm
- net /DRIVER1/STEP: track 0.00 -> 14.2 mm
- net VMOT: track 175.0 -> 169.1 mm
- net /DRIVER3/nENBL: track 39.5 -> 40.9 mm
- net /DRIVER3/MODE0: track 45.9 -> 45.0 mm
- net /DRIVER3/CURR_REF: track 70.8 -> 71.6 mm
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
Commit message: 4 kesz
Routing:
- net 3.3V: track 403.7 -> 550.7 mm
- net /DRIVER1/CURR_REF: track 0.00 -> 74.8 mm
- net VMOT: track 169.1 -> 226.2 mm
- net /DRIVER1/nFAULT: track 23.3 -> 77.7 mm, vias 0 -> 1
- net /DRIVER1/AOUT1: track 0.00 -> 53.4 mm, vias 0 -> 1
- net /DRIVER1/AOUT2: track 0.00 -> 48.0 mm, vias 0 -> 1
- net /DRIVER1/nHOME: track 24.4 -> 68.7 mm, vias 0 -> 1
- net /DRIVER1/MODE2: track 23.4 -> 62.5 mm, vias 0 -> 1
- net /DRIVER1/DIR: track 15.2 -> 52.8 mm, vias 0 -> 1
- net /DRIVER1/BOUT2: track 0.00 -> 35.3 mm, vias 0 -> 1
- net Net-(D2-Pad1): track 0.00 -> 34.5 mm, vias 0 -> 2
- net /DRIVER1/MODE1: track 22.5 -> 56.5 mm, vias 0 -> 1
- net /DRIVER1/MODE0: track 21.5 -> 52.4 mm, vias 0 -> 1
- net /DRIVER1/BOUT1: track 0.00 -> 30.6 mm, vias 0 -> 1
- net Net-(P8-Pad2): track 0.00 -> 30.0 mm, vias 0 -> 1
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
Commit message: trafo bent
Parts:
- P1: value UART_HEAD -> CONN_01X04; footprint libs:PIN_CONN_0.3Inch -> Pin_Headers:Pin_Header_Straight_1x04
- P3: value PROG_HEAD -> CONN_01X04; footprint libs:PIN_CONN_0.3Inch -> Pin_Headers:Pin_Header_Straight_1x04
- moved C6 534.1 mm to (555.2, 192.6), turned to 90 degrees
- moved C5 496.2 mm to (531.2, 192.8), turned to 90 degrees
- moved P19 494.3 mm to (595.0, 185.8), turned to 180 degrees
- moved P2 438.8 mm to (460.3, 187.6), turned to 180 degrees
- moved P6 430.6 mm to (512.2, 194.4)
- moved P4 402.2 mm to (399.4, 198.5), turned to 90 degrees
- moved C1 395.8 mm to (464.1, 136.7)
- moved R13 395.8 mm to (487.2, 132.6)
- moved R14 395.8 mm to (495.2, 122.3)
- moved R16 395.8 mm to (478.2, 138.3)
- moved R3 395.8 mm to (471.1, 138.3)
- moved R4 395.8 mm to (487.2, 125.9)
- moved R6 395.8 mm to (485.2, 139.3)
- moved C7 391.7 mm to (500.0, 148.8)
- moved R11 391.7 mm to (514.1, 144.7)
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Connections:
- C4 pad 2: GND -> VMOT_GND
- C5 pad 2: GND -> VMOT_GND
- C6 pad 2: GND -> VMOT_GND
- C7 pad 2: GND -> VMOT_GND
- P1 pad 1: Net-(P1-Pad1) -> GND
- P3 pad 1: Net-(P3-Pad1) -> GND
- P6 pad 2: GND -> VMOT_GND
- R17 pad 1: Net-(P3-Pad2) -> Net-(P3-Pad3)
- R19 pad 2: GND -> VMOT_GND
- R20 pad 2: GND -> VMOT_GND
- R31 pad 2: GND -> VMOT_GND
- R32 pad 2: GND -> VMOT_GND
- R43 pad 2: GND -> VMOT_GND
- R44 pad 2: GND -> VMOT_GND
- R55 pad 2: GND -> VMOT_GND
- R56 pad 2: GND -> VMOT_GND
- U1 pad 16: Net-(P3-Pad2) -> Net-(P3-Pad3)
- U1 pad 17: Net-(P3-Pad1) -> Net-(P3-Pad2)
- U1 pad 20: Net-(U1-Pad20) -> GND
- U1 pad 3: Net-(P1-Pad2) -> Net-(P1-Pad3)
- U1 pad 4: Net-(P1-Pad1) -> Net-(P1-Pad2)
Routing:
- net 3.3V: track 550.7 -> 669.4 mm, vias 1 -> 3
- net Net-(P2-Pad2): track 0.00 -> 95.4 mm, vias 0 -> 1
- net Net-(C11-Pad1): track 0.00 -> 89.4 mm, vias 0 -> 1
- net Net-(D1-Pad2): track 0.00 -> 41.4 mm
- net Net-(P3-Pad3): track 0.00 -> 39.7 mm
- net Net-(P3-Pad2): track 0.00 -> 38.3 mm
- net Net-(P1-Pad2): track 0.00 -> 38.3 mm
- net Net-(P1-Pad3): track 0.00 -> 36.4 mm
- net Net-(D1-Pad4): track 0.00 -> 30.8 mm
- net Net-(P5-Pad1): track 0.00 -> 24.6 mm
- net Net-(P5-Pad2): track 0.00 -> 22.1 mm
- net /MOSI: track 0.00 -> 18.5 mm
- net /DRIVER1/STEP: track 40.4 -> 57.3 mm
- net VMOT_GND: track 0.00 -> 9.77 mm, vias 0 -> 2
- net /PIN3: track 0.00 -> 7.75 mm
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Other:
- net class Default: clearance 0.3048 -> 0.254
- rule trace_clearance: 0.3048 -> 0.254
