File: semCNC.sch (KiCad schematic (older format))
At the start: 42 parts, among them P1 CONN_01X04, P19 POWER_HEAD, P2 LPT port, P3 CONN_01X04, P4 EXPANDER PAD, P5 CONN_01X02, P6 CONN_01X02, T1 TRANSFO, U1 MSP430G2452, U2 TIdac08s085, U3 LD1117S33CTR, U4 SPX2920U-3.3

Commit message: mer elegem van .... :P
Parts:
- added P20: CONN_01X02, Pin_Headers:Pin_Header_Straight_1x02, symbol CONN_01X02
Connections:
- wire segments 123 -> 125
Changed lines of the file:
@@
 	1    0    0    -1
 $EndComp
+$Comp
+L CONN_01X02 P20
+U 1 1 561E9201
+P 8650 1200
+F 0 "P20" H 8650 1350 50  0000 C CNN
+F 1 "CONN_01X02" V 8750 1200 50  0000 C CNN
+F 2 "Pin_Headers:Pin_Header_Straight_1x02" H 8650 1200 60  0001 C CNN
+F 3 "" H 8650 1200 60  0000 C CNN
+	1    8650 1200
+	1    0    0    -1
+$EndComp
+$Comp
+L Earth #PWR035
+U 1 1 561E9402
+P 8450 1250
+F 0 "#PWR035" H 8450 1000 50  0001 C CNN
+F 1 "Earth" H 8450 1100 50  0001 C CNN
+F 2 "" H 8450 1250 60  0000 C CNN
+F 3 "" H 8450 1250 60  0000 C CNN
+	1    8450 1250
+	0    1    1    0
+$EndComp
+Wire Wire Line
+	8350 900  8350 1150
+Wire Wire Line
+	8350 1150 8450 1150
 $EndSCHEMATC

Commit message: New layout
Parts:
- added P21: CONN_01X02, Pin_Headers:Pin_Header_Straight_1x02, symbol CONN_01X02
Changed lines of the file:
@@
 LIBS:contrib
 LIBS:valves
+LIBS:mylib
 LIBS:semCNC-cache
 EELAYER 25 0
@@
 Text Label 5850 3950 0    60   ~ 0
 IREF4
+Text Label 5850 2450 0    60   ~ 0
+IREF3
 Text Label 5850 3200 0    60   ~ 0
-IREF3
-Text Label 5850 2450 0    60   ~ 0
 IREF2
 Text Label 5850 1650 0    60   ~ 0
@@
 Text Label 5850 3750 0    60   ~ 0
 STEP4
+Text Label 5850 2550 0    60   ~ 0
+nFAULT3
+Text Label 5850 2350 0    60   ~ 0
+DIR3
+Text Label 5850 2250 0    60   ~ 0
+STEP3
 Text Label 5850 3300 0    60   ~ 0
-nFAULT3
+nFAULT2
 Text Label 5850 3100 0    60   ~ 0
-DIR3
+DIR2
 Text Label 5850 3000 0    60   ~ 0
-STEP3
-Text Label 5850 2550 0    60   ~ 0
-nFAULT2
-Text Label 5850 2350 0    60   ~ 0
-DIR2
-Text Label 5850 2250 0    60   ~ 0
 STEP2
 Text Label 5850 1750 0    60   ~ 0
@@
 Text Label 5850 1450 0    60   ~ 0
 STEP1
+Text Label 3150 3100 0    60   ~ 0
+STEP4
+Text Label 3150 3300 0    60   ~ 0
+STEP3
+Text Label 3150 3400 0    60   ~ 0
+STEP2
 Text Label 3150 3500 0    60   ~ 0
-STEP4
-Text Label 3150 3400 0    60   ~ 0
-STEP3
-Text Label 3150 3300 0    60   ~ 0
-STEP2
-Text Label 3150 3100 0    60   ~ 0
 STEP1
 Text Label 1000 3500 0    60   ~ 0
@@
 L Earth #PWR027
 U 1 1 56065958
-P 3200 1000
-F 0 "#PWR027" H 3200 750 50  0001 C CNN
-F 1 "Earth" H 3200 850 50  0001 C CNN
-F 2 "" H 3200 1000 60  0000 C CNN
-F 3 "" H 3200 1000 60  0000 C CNN
-	1    3200 1000
+P 3200 1100
+F 0 "#PWR027" H 3200 850 50  0001 C CNN
+F 1 "Earth" H 3200 950 50  0001 C CNN
+F 2 "" H 3200 1100 60  0000 C CNN
+F 3 "" H 3200 1100 60  0000 C CNN
+	1    3200 1100
 	1    0    0    -1
 $EndComp
@@
 Wire Wire Line
 	8350 1150 8450 1150
+$Comp
+L CONN_01X02 P21
+U 1 1 562419D1
+P 3400 1050
+F 0 "P21" H 3400 1200 50  0000 C CNN
+F 1 "CONN_01X02" V 3500 1050 50  0000 C CNN
+F 2 "Pin_Headers:Pin_Header_Straight_1x02" H 3400 1050 60  0001 C CNN
+F 3 "" H 3400 1050 60  0000 C CNN
+	1    3400 1050
+	1    0    0    -1
+$EndComp
 $EndSCHEMATC

Commit message: minor changes in layout
Parts:
- removed C3: C, Capacitors_SMD:C_1206_HandSoldering, symbol C
- removed U2: TIdac08s085, libs:TI_VSSOP10_DGS, symbol TIdac08s085
- added U2: ANALOG_DEVICES_AD7304, Housings_SOIC:SOIC-16_7.5x10.3mm_Pitch1.27mm, symbol ANALOG_DEVICES_AD7304
- D1: symbol Diode_Bridge -> Diode_Bridge-RESCUE-semCNC
Connections:
- wire segments 125 -> 109
